File: Arduino-Pro-Mini-v13.brd (EAGLE design)
At the start: 17.8 x 33 mm, 20 parts, among them Q1 8/16/20MHz, U1 ATMEGA328, U2 MIC5205

Commit message: Removed
Parts:
- removed JP5, JP8: FIDUCIALUFIDUCIAL, SparkFun:MICRO-FIDUCIAL
- added FRM1: (no value), Frames:LETTER
Other:
- board text removed: "Released under the Creative Commons Attribution Share-Alike 3.0 License"
- board text removed: "http://creativecommons.org/licenses/by-sa/3.0"
Changed lines of the file:
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@@
 <text x="1.27" y="30.734" size="0.8128" layer="21" ratio="15" rot="R90">BLK</text>
 <text x="17.272" y="30.734" size="0.8128" layer="21" ratio="15" rot="R90">GRN</text>
-<text x="-43.18" y="-5.08" size="1.778" layer="21">Released under the Creative Commons Attribution Share-Alike 3.0 License</text>
-<text x="-25.4" y="-7.62" size="1.778" layer="21">http://creativecommons.org/licenses/by-sa/3.0</text>
 <text x="19.812" y="26.162" size="1.27" layer="27">Valid combinations:</text>
 <text x="19.812" y="23.622" size="1.27" layer="27">168V / 3.3V Reg / 8MHz</text>
@@
 <element name="JP1" library="SparkFun" package="1X06" value="FTDI Basic" x="15.24" y="31.75" rot="MR0"/>
 <element name="C2" library="SparkFun" package="0402-CAP" value="0.1uF" x="12.8016" y="29.21" rot="R180"/>
-<element name="JP5" library="SparkFun" package="MICRO-FIDUCIAL" value="FIDUCIALUFIDUCIAL" x="4.064" y="28.956"/>
-<element name="JP8" library="SparkFun" package="MICRO-FIDUCIAL" value="FIDUCIALUFIDUCIAL" x="12.446" y="2.54"/>
+<element name="FRM1" library="Frames" package="LETTER" value="" x="-7.62" y="-3.81"/>
 </elements>
 <signals>
