File: Arduino-Pro-Mini-v13.sch (EAGLE design)
At the start: 20 parts, among them Q1 8/16/20MHz, U1 ATMEGA328, U2 MIC5205

Commit message: Removed
Parts:
- removed JP5, JP8: FIDUCIALUFIDUCIAL, SparkFun:FIDUCIALUFIDUCIAL
- added FRM1: (no value), Frames:LETTER
Other:
- note removed: "Arduino Pro Mini Design by Spark Fun Electronics"
- note removed: "Board is marked with combination of"
- note removed: "Original Arduino Mini Design by Team Arduino"
- note removed: "Released under the Creative Commons Attribution Share-Alike 3.0 License"
- note removed: "http://creativecommons.org/licenses/by-sa/3.0"
- note removed: "resonator frequency and regulator voltage."
Changed lines of the file:
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@@
 <parts>
 <part name="C10" library="SparkFun" deviceset="CAP" device="0402-CAP" value="0.1uF"/>
-<part name="FRAME1" library="SparkFun" deviceset="FRAME-LETTER" device=""/>
 <part name="C13" library="SparkFun" deviceset="CAP_POL" device="1206" value="10uF"/>
 <part name="GND25" library="SparkFun" deviceset="GND" device=""/>
@@
 <part name="P+2" library="SparkFun" deviceset="3.3V" device="" value="VCC"/>
 <part name="P+3" library="SparkFun" deviceset="3.3V" device="" value="VCC"/>
-<part name="JP5" library="SparkFun" deviceset="FIDUCIAL" device="UFIDUCIAL"/>
-<part name="JP8" library="SparkFun" deviceset="FIDUCIAL" device="UFIDUCIAL"/>
+<part name="FRM1" library="Frames" deviceset="LETTER" device=""/>
 </parts>
 <sheets>
 <sheet>
 <plain>
-<wire x1="53.34" y1="58.42" x2="53.34" y2="30.48" width="0.2032" layer="97" style="shortdash"/>
-<text x="17.78" y="17.78" size="1.778" layer="95">Released under the Creative Commons Attribution Share-Alike 3.0 License</text>
-<text x="17.78" y="15.24" size="1.778" layer="95">http://creativecommons.org/licenses/by-sa/3.0</text>
-<text x="17.78" y="10.16" size="1.778" layer="95">Original Arduino Mini Design by Team Arduino</text>
-<text x="17.78" y="7.62" size="1.778" layer="95">Arduino Pro Mini Design by Spark Fun Electronics</text>
 <text x="35.56" y="137.16" size="1.778" layer="97">Max Voltage Input: 16VDC</text>
 <text x="35.56" y="134.62" size="1.778" layer="97">Max Current Output: 150mA</text>
-<text x="27.94" y="124.46" size="1.778" layer="97">Board is marked with combination of</text>
-<text x="22.86" y="121.92" size="1.778" layer="97">resonator frequency and regulator voltage.</text>
 <text x="35.56" y="139.7" size="1.778" layer="97">VCC = 5V or 3.3V Output</text>
 <text x="259.08" y="182.88" size="1.778" layer="94">Changes to v13 (10-12-11)</text>
@@
 <instances>
 <instance part="C10" gate="G$1" x="66.04" y="154.94"/>
-<instance part="FRAME1" gate="G$1" x="0" y="0"/>
-<instance part="FRAME1" gate="G$2" x="147.32" y="0"/>
 <instance part="C13" gate="G$1" x="58.42" y="157.48"/>
 <instance part="GND25" gate="1" x="58.42" y="147.32"/>
@@
 <instance part="P+2" gate="G$1" x="223.52" y="160.02"/>
 <instance part="P+3" gate="G$1" x="231.14" y="160.02"/>
-<instance part="JP5" gate="G$1" x="238.76" y="27.94"/>
-<instance part="JP8" gate="G$1" x="238.76" y="33.02"/>
+<instance part="FRM1" gate="FRAME" x="0" y="0"/>
+<instance part="FRM1" gate="DOCFIELDS" x="152.4" y="0"/>
 </instances>
 <busses>
